Commit message: add lidar sensor to kobuki gazebo model

File: kobuki_description/urdf/kobuki.urdf.xacro (robot description, xacro)
@@ -208,4 +208,31 @@
       </inertial>
     </link>
+    <joint name="scan_joint" type="fixed">
+      <parent link="base_link"/>
+      <child link="base_scan"/>
+      <origin xyz="0 0 0.15" rpy="0 0 0"/>
+    </joint>
+    <link name="base_scan">
+      <visual>
+        <origin xyz="0 0 0" rpy="0 0 0"/>
+        <geometry>
+          <mesh filename="package://kobuki_description/meshes/sensors/lds.stl" scale="0.001 0.001 0.001"/>
+        </geometry>
+        <material name="dark"/>
+      </visual>
+      <collision>
+        <origin xyz="0.015 0 -0.0065" rpy="0 0 0"/>
+        <geometry>
+          <cylinder length="0.0315" radius="0.055"/>
+        </geometry>
+      </collision>
+      <inertial>
+        <mass value="0.114" />
+        <origin xyz="0 0 0" />
+        <inertia ixx="0.001" ixy="0.0" ixz="0.0"
+                 iyy="0.001" iyz="0.0"
+                 izz="0.001" />
+      </inertial>
+    </link>
     <!-- Kobuki Gazebo simulation details -->
     <xacro:kobuki_sim/>

File: kobuki_description/urdf/kobuki_gazebo.urdf.xacro (robot description, xacro)
@@ -160,4 +160,36 @@
       </sensor>
 	  </gazebo>
+	  <gazebo reference="base_scan">
+		  <material>Gazebo/FlatBlack</material>
+		  <sensor type="ray" name="lds_lfcd_sensor">
+			  <pose>0 0 0 0 0 0</pose>
+			  <visualize>true</visualize>
+			  <update_rate>5</update_rate>
+			  <ray>
+				  <scan>
+					  <horizontal>
+						  <samples>360</samples>
+						  <resolution>1</resolution>
+						  <min_angle>0.0</min_angle>
+						  <max_angle>6.28319</max_angle>
+					  </horizontal>
+				  </scan>
+				  <range>
+					  <min>0.120</min>
+					  <max>3.5</max>
+					  <resolution>0.015</resolution>
+				  </range>
+				  <noise>
+					  <type>gaussian</type>
+					  <mean>0.0</mean>
+					  <stddev>0.01</stddev>
+				  </noise>
+			  </ray>
+			  <plugin name="gazebo_ros_lds_lfcd_controller" filename="libgazebo_ros_laser.so">
+				  <topicName>scan</topicName>
+				  <frameName>base_scan</frameName>
+			  </plugin>
+		  </sensor>
+	  </gazebo>
 	  <gazebo>
 	    <plugin name="kobuki_controller" filename="libgazebo_ros_kobuki.so">
